Commit message: Added a file to run the comparison between the model obtained by applying the optimization method and the real one of the LoCoBot WX250s

File: generate_pointcloud/model/mobile_wx250s.urdf (robot description, URDF)
Before this commit: robot mobile_wx250s, 15 links, 14 joints
Links:
- link locobot/ar_tag_link: geometry collision mesh filename=/home/rosario/Desktop/Robotic-manipulators-reachability-spa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 scale=0.001 0.001 0.001; visual mesh filename=/home/rosario/Desktop/Robotic-manipulators-reachability-spa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 scale=0.001 0.001 0.001
- link locobot/arm_base_link: geometry collision mesh filename=/home/rosario/Desktop/Robotic-manipulators-reachability-spa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 scale=0.001 0.001 0.001; visual mesh filename=/home/rosario/Desktop/Robotic-manipulators-reachability-spa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 scale=0.001 0.001 0.001
- link locobot/gripper_bar_link: geometry collision mesh filename=/home/rosario/Desktop/Robotic-manipulators-reachability-spa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 scale=0.001 0.001 0.001; visual mesh filename=/home/rosario/Desktop/Robotic-manipulators-reachability-spa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 scale=0.001 0.001 0.001
- link locobot/gripper_link: geometry collision mesh filename=/home/rosario/Desktop/Robotic-manipulators-reachability-spa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 scale=0.001 0.001 0.001; visual mesh filename=/home/rosario/Desktop/Robotic-manipulators-reachability-spa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 scale=0.001 0.001 0.001
- link locobot/gripper_prop_link: geometry collision mesh filename=/home/rosario/Desktop/Robotic-manipulators-reachability-spa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 scale=0.001 0.001 0.001; visual mesh filename=/home/rosario/Desktop/Robotic-manipulators-reachability-spa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 scale=0.001 0.001 0.001
- link locobot/left_finger_link: geometry collision mesh filename=/home/rosario/Desktop/Robotic-manipulators-reachability-spa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 scale=0.001 0.001 0.001; visual mesh filename=/home/rosario/Desktop/Robotic-manipulators-reachability-spa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 scale=0.001 0.001 0.001
- link locobot/lower_forearm_link: geometry collision mesh filename=/home/rosario/Desktop/Robotic-manipulators-reachability-spa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 scale=0.001 0.001 0.001; visual mesh filename=/home/rosario/Desktop/Robotic-manipulators-reachability-spa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 scale=0.001 0.001 0.001
- link locobot/right_finger_link: geometry collision mesh filename=/home/rosario/Desktop/Robotic-manipulators-reachability-spa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 scale=0.001 0.001 0.001; visual mesh filename=/home/rosario/Desktop/Robotic-manipulators-reachability-spa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 scale=0.001 0.001 0.001
- link locobot/shoulder_link: geometry collision mesh filename=/home/rosario/Desktop/Robotic-manipulators-reachability-spa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 scale=0.001 0.001 0.001; visual mesh filename=/home/rosario/Desktop/Robotic-manipulators-reachability-spa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 scale=0.001 0.001 0.001
- link locobot/upper_arm_link: geometry collision mesh filename=/home/rosario/Desktop/Robotic-manipulators-reachability-spa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 scale=0.001 0.001 0.001; visual mesh filename=/home/rosario/Desktop/Robotic-manipulators-reachability-spa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 scale=0.001 0.001 0.001
- link locobot/upper_forearm_link: geometry collision mesh filename=/home/rosario/Desktop/Robotic-manipulators-reachability-spa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 scale=0.001 0.001 0.001; visual mesh filename=/home/rosario/Desktop/Robotic-manipulators-reachability-spa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 scale=0.001 0.001 0.001
- link locobot/wrist_link: geometry collision mesh filename=/home/rosario/Desktop/Robotic-manipulators-reachability-spa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 scale=0.001 0.001 0.001; visual mesh filename=/home/rosario/Desktop/Robotic-manipulators-reachability-spa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 scale=0.001 0.001 0.001
